Commit message: Ekuthon

File: ur_e_description/urdf/ur5e.urdf.xacro (robot description, xacro)
@@ -344,9 +344,9 @@
     </joint>
     <!-- Frame coincident with all-zeros TCP on UR controller -->
-    <link name="${prefix}tool0"/>
+    <!-- <link name="${prefix}palm"/> -->
     <joint name="${prefix}wrist_3_link-tool0_fixed_joint" type="fixed">
-      <origin xyz="0 ${wrist_3_length} 0" rpy="${pi/-2.0} 0 0"/>
+      <origin xyz="0 ${wrist_3_length} 0" rpy="0 0 0"/>
       <parent link="${prefix}wrist_3_link"/>
-      <child link="${prefix}tool0"/>
+      <child link="${prefix}palm"/>
     </joint>
   </xacro:macro>

File: ur_e_description/urdf/ur5e_joint_limited_robot.urdf.xacro (robot description, xacro)
@@ -15,9 +15,12 @@
     wrist_3_lower_limit="${-pi}" wrist_3_upper_limit="${pi}"
   />
-  <link name="world" />
-  <joint name="world_joint" type="fixed">
-    <parent link="world" />
+  <!--
+    Renamed link:
+    https://github.com/ros-industrial/universal_robot/pull/284
+    -->
+  <link name="robot_base" />
+  <joint name="robot_base_joint" type="fixed">
+    <parent link="robot_base" />
     <child link = "base_link" />
-    <origin xyz="0.0 0.0 0.0" rpy="0.0 0.0 0.0" />
   </joint>
 </robot>
